Commit message: Update the xacros
Signed-off-by: Christoph Hellmann Santos <christoph.hellmann.santos@ipa.fraunhofer.de>

File: ur5e_cell_description/urdf/robot_cell.xacro (robot description, xacro)
@@ -1,122 +1,124 @@
 <?xml version="1.0"?>
-<robot xmlns:xacro="http://www.ros.org/wiki/xacro">
+<robot xmlns:xacro="http://www.ros.org/wiki/xacro" name="robot_cell">
     <xacro:include filename="inertial_macros.xacro"/>
-    <xacro:property name="robot_center_offset_length" value="0.42" />
-    <xacro:property name="robot_center_offset_width" value="0.02" />
-    <xacro:property name="robot_base_height" value="0.99" />
-    <xacro:property name="robotcell_length" value="1.44" />
-    <xacro:property name="robotcell_width" value="0.94" />
-    <xacro:property name="robotcell_height" value="1.16" />
-    <xacro:property name="shield_thickness" value="0.03" />
-    <material name="gray">
-        <color rgba="0.6 0.8 0.8 1" />
-    </material>
-    <link name="shield_front_link">
-        <collision>
-            <origin rpy="0 0 0" xyz="0 0 0" />
-            <geometry>
-                <box size="${robotcell_length} ${shield_thickness} ${robotcell_height}" />
-            </geometry>
-            <material name="gray"/>
-        </collision>
-        <xacro:inertial_box mass="5" x="${robotcell_length}" y="${shield_thickness}" z="${robotcell_height}">
-            <origin rpy="0 0 0" xyz="0 0 0" />
-        </xacro:inertial_box>
-    </link>
-    <link name="shield_rear_link">
-        <visual>
-            <origin rpy="0 0 0" xyz="0 0 0" />
-            <geometry>
-                <box size="${robotcell_length} ${shield_thickness} ${robotcell_height}" />
-            </geometry>
-            <material name="gray"/>
-        </visual>
-        <collision>
-            <origin rpy="0 0 0 " xyz="0 0 0" />
-            <geometry>
-                <box size="${robotcell_length} ${shield_thickness} ${robotcell_height}" />
-            </geometry>
-            <material name="gray"/>
-        </collision>
-        <xacro:inertial_box mass="5" x="${robotcell_length}" y="${shield_thickness}" z="${robotcell_height}">
-            <origin rpy="0 0 0" xyz="0 0 0" />
-        </xacro:inertial_box>
-    </link>
-    <link name="shield_right_link">
-        <visual>
-            <origin rpy="0 0 0" xyz="0 0 0" />
-            <geometry>
-                <box size="${shield_thickness} ${robotcell_width} ${robotcell_height}" />
-            </geometry>
-            <material name="gray"/>
-        </visual>
-        <collision>
-            <origin rpy="0 0 0" xyz="0 0 0" />
-            <geometry>
-                <box size="${shield_thickness} ${robotcell_width} ${robotcell_height}" />
-            </geometry>
-            <material name="gray"/>
-        </collision>
-        <xacro:inertial_box mass="5" x="${shield_thickness}" y="${robotcell_width}" z="${robotcell_height}">
-            <origin rpy="0 0 0" xyz="0 0 0" />
-        </xacro:inertial_box>
-    </link>
-    <link name="shield_left_link">
-        <visual>
-            <origin rpy="0 0 0" xyz="0 0 0" />
-            <geometry>
-                <box size="${shield_thickness} ${robotcell_width} ${robotcell_height}" />
-            </geometry>
-            <material name="gray"/>
-        </visual>
-        <collision>
-            <origin rpy="0 0 0" xyz="0 0 0" />
-            <geometry>
-                <box size="${shield_thickness} ${robotcell_width} ${robotcell_height}" />
-            </geometry>
-            <material name="gray"/>
-        </collision>
-        <xacro:inertial_box mass="5" x="${shield_thickness}" y="${robotcell_width}" z="${robotcell_height}">
-            <origin rpy="0 0 0" xyz="0 0 0" />
-        </xacro:inertial_box>
-    </link>
-    <link name="robotcell_base_link">
-        <visual>
-            <origin rpy="0 0 0" xyz="0 0 ${robot_base_height/2}" />
-            <geometry>
-                <box size="${robotcell_length} ${robotcell_width} ${robot_base_height}" />
-            </geometry>
-            <material name="gray"/>
-        </visual>
-        <collision>
-            <origin rpy="0 0 0" xyz="0 0 ${robot_base_height/2}" />
-            <geometry>
-                <box size="${robotcell_length} ${robotcell_width} ${robot_base_height}" />
-            </geometry>
-            <material name="gray"/>
-        </collision>
-        <xacro:inertial_box mass="70" x="${robotcell_length}" y="${robotcell_width}" z="${robot_base_height}">
-            <origin rpy="0 0 0" xyz="0 0 0" />
-        </xacro:inertial_box>
-    </link>
-    <joint name="robotcell_base_to_front_joint" type="fixed">
-        <parent link="robotcell_base_link" />
-        <child link="shield_front_link" />
-        <origin xyz="0 ${robotcell_width/2-shield_thickness/2} ${robot_base_height+robotcell_height/2}" rpy="0 0 0" />
-    </joint>
-    <joint name="robotcell_base_to_rear" type="fixed">
-        <parent link="robotcell_base_link" />
-        <child link="shield_rear_link" />
-        <origin xyz="0 ${-robotcell_width/2+shield_thickness/2} ${robot_base_height+robotcell_height/2}" rpy="0 0 0" />
-    </joint>
-    <joint name="robotcell_base_to_left" type="fixed">
-        <parent link="robotcell_base_link" />
-        <child link="shield_left_link" />
-        <origin xyz="${-robotcell_length/2+shield_thickness/2} 0 ${robot_base_height+robotcell_height/2}" rpy="0 0 0" />
-    </joint>
-    <joint name="robotcell_jbase_to_right" type="fixed">
-        <parent link="robotcell_base_link" />
-        <child link="shield_right_link" />
-        <origin xyz="${robotcell_length/2-shield_thickness/2} 0 ${robot_base_height+robotcell_height/2}" rpy="0 0 0" />
-    </joint>
+    <xacro:macro name="robot_cell" params="
+        name
+        prefix
+        parent
+        *origin">
+        <xacro:property name="robot_center_offset_length" value="0.42" />
+        <xacro:property name="robot_center_offset_width" value="0.02" />
+        <xacro:property name="robot_base_height" value="0.99" />
+        <xacro:property name="robotcell_length" value="1.44" />
+        <xacro:property name="robotcell_width" value="0.94" />
+        <xacro:property name="robotcell_height" value="1.16" />
+        <xacro:property name="shield_thickness" value="0.03" />
+        <material name="gray">
+            <color rgba="0.6 0.8 0.8 1" />
+        </material>
+        <link name="${prefix}visuals_link">
+            <visual>
+                <geometry>
+                    <mesh filename="package://ur5e_cell_description/meshes/Assembly_new.STL" scale="0.001 0.001 0.001" />
+                </geometry>
+                <material name="gray"/>
+            </visual>
+        </link>
+        <link name="${prefix}shield_front_link">
+            <collision>
+                <origin rpy="0 0 0" xyz="0 0 0" />
+                <geometry>
+                    <box size="${robotcell_length} ${shield_thickness} ${robotcell_height}" />
+                </geometry>
+                <material name="gray"/>
+            </collision>
+            <xacro:inertial_box mass="5" x="${robotcell_length}" y="${shield_thickness}" z="${robotcell_height}">
+                <origin rpy="0 0 0" xyz="0 0 0" />
+            </xacro:inertial_box>
+        </link>
+        <link name="${prefix}shield_rear_link">
+            <collision>
+                <origin rpy="0 0 0 " xyz="0 0 0" />
+                <geometry>
+                    <box size="${robotcell_length} ${shield_thickness} ${robotcell_height}" />
+                </geometry>
+                <material name="gray"/>
+            </collision>
+            <xacro:inertial_box mass="5" x="${robotcell_length}" y="${shield_thickness}" z="${robotcell_height}">
+                <origin rpy="0 0 0" xyz="0 0 0" />
+            </xacro:inertial_box>
+        </link>
+        <link name="${prefix}shield_right_link">
+            <collision>
+                <origin rpy="0 0 0" xyz="0 0 0" />
+                <geometry>
+                    <box size="${shield_thickness} ${robotcell_width} ${robotcell_height}" />
+                </geometry>
+                <material name="gray"/>
+            </collision>
+            <xacro:inertial_box mass="5" x="${shield_thickness}" y="${robotcell_width}" z="${robotcell_height}">
+                <origin rpy="0 0 0" xyz="0 0 0" />
+            </xacro:inertial_box>
+        </link>
+        <link name="${prefix}shield_left_link">
+            <collision>
+                <origin rpy="0 0 0" xyz="0 0 0" />
+                <geometry>
+                    <box size="${shield_thickness} ${robotcell_width} ${robotcell_height}" />
+                </geometry>
+                <material name="gray"/>
+            </collision>
+            <xacro:inertial_box mass="5" x="${shield_thickness}" y="${robotcell_width}" z="${robotcell_height}">
+                <origin rpy="0 0 0" xyz="0 0 0" />
+            </xacro:inertial_box>
+        </link>
+        <link name="${prefix}robotcell_base_link">
+            <collision>
+                <origin rpy="0 0 0" xyz="0 0 ${robot_base_height/2}" />
+                <geometry>
+                    <box size="${robotcell_length} ${robotcell_width} ${robot_base_height}" />
+                </geometry>
+                <material name="gray"/>
+            </collision>
+            <xacro:inertial_box mass="70" x="${robotcell_length}" y="${robotcell_width}" z="${robot_base_height}">
+                <origin rpy="0 0 0" xyz="0 0 0" />
+            </xacro:inertial_box>
+        </link>
+        <link name="${prefix}robot_link" />
+        <joint name="${prefix}robotcell_base_to_visual" type="fixed">
+            <parent link="${prefix}robotcell_base_link" />
+            <child link="${prefix}visuals_link" />
+            <origin xyz="${robotcell_length/2+shield_thickness} -${robotcell_width/2+shield_thickness} 0" rpy="0 0 ${pi/2}" />
+        </joint>
+        <joint name="${prefix}robotcell_base_to_front_joint" type="fixed">
+            <parent link="${prefix}robotcell_base_link" />
+            <child link="${prefix}shield_front_link" />
+            <origin xyz="0 ${robotcell_width/2-shield_thickness/2} ${robot_base_height+robotcell_height/2}" rpy="0 0 0" />
+        </joint>
+        <joint name="${prefix}robotcell_base_to_rear" type="fixed">
+            <parent link="${prefix}robotcell_base_link" />
+            <child link="${prefix}shield_rear_link" />
+            <origin xyz="0 ${-robotcell_width/2+shield_thickness/2} ${robot_base_height+robotcell_height/2}" rpy="0 0 0" />
+        </joint>
+        <joint name="${prefix}robotcell_base_to_left" type="fixed">
+            <parent link="${prefix}robotcell_base_link" />
+            <child link="${prefix}shield_left_link" />
+            <origin xyz="${-robotcell_length/2+shield_thickness/2} 0 ${robot_base_height+robotcell_height/2}" rpy="0 0 0" />
+        </joint>
+        <joint name="${prefix}robotcell_base_to_right" type="fixed">
+            <parent link="${prefix}robotcell_base_link" />
+            <child link="${prefix}shield_right_link" />
+            <origin xyz="${robotcell_length/2-shield_thickness/2} 0 ${robot_base_height+robotcell_height/2}" rpy="0 0 0" />
+        </joint>
+        <joint name="${prefix}robot_cell_base_joint" type="fixed">
+            <parent link="${parent}" />
+            <child link="${prefix}robotcell_base_link" />
+            <xacro:insert_block name="origin" />
+        </joint>
+        <joint name="${prefix}robot_cell_base_to_robot_link" type="fixed">
+            <parent link="${prefix}robotcell_base_link" />
+            <child link="${prefix}robot_link" />
+            <origin xyz="${robot_center_offset_length} ${robot_center_offset_width} ${robot_base_height}" rpy="0 0 0" />
+        </joint>
+    </xacro:macro>
 </robot>

File: ur5e_cell_description/urdf/schunk_egp50.xacro (robot description, xacro)
@@ -1,5 +1,10 @@
 <?xml version="1.0"?>
 <robot xmlns:xacro="http://www.ros.org/wiki/xacro" name="schunk_egp50">
-    <xacro:macro name="schunk_egp50">
+    <xacro:macro name="schunk_egp50" params="
+        name
+        prefix
+        parent
+        *origin
+    ">
         <xacro:include filename="inertial_macros.xacro" />
         <xacro:property name="base_diameter" value="0.075" />
@@ -22,5 +27,5 @@
         </material>
         <!--Base plate-->
-        <link name="shunk_egp50_base_link">
+        <link name="${prefix}schunk_egp50_base_link">
             <visual>
                 <geometry>
@@ -41,5 +46,5 @@
         </link>
         <!--Main gripper-->
-        <link name="shunk_egp50_body_link">
+        <link name="${prefix}schunk_egp50_body_link">
             <visual>
                 <geometry>
@@ -60,5 +65,5 @@
         </link>
         <!--Pincer block 1-->
-        <link name="shunk_egp50_pincer_1_link">
+        <link name="${prefix}schunk_egp50_pincer_1_link">
             <visual>
                 <geometry>
@@ -79,5 +84,5 @@
         </link>
         <!--Pincer block 2-->
-        <link name="shunk_egp50_pincer_2_link">
+        <link name="${prefix}schunk_egp50_pincer_2_link">
             <visual>
                 <geometry>
@@ -100,12 +105,12 @@
         <link name="tool_tip" />
         <!-- Joints-->
-        <joint name="shunk_egp50_body_joint" type="fixed">
-            <parent link="shunk_egp50_base_link" />
-            <child link="shunk_egp50_body_link" />
+        <joint name="${prefix}schunk_egp50_body_joint" type="fixed">
+            <parent link="${prefix}schunk_egp50_base_link" />
+            <child link="${prefix}schunk_egp50_body_link" />
             <origin xyz="0.0 0.0 ${base_length+body_height/2}" rpy="0.0 0.0 0.0" />
         </joint>
-        <joint name="shunk_egp50_pincer_1_joint" type="fixed">
-            <parent link="shunk_egp50_body_link" />
-            <child link="shunk_egp50_pincer_1_link" />
+        <joint name="${prefix}schunk_egp50_pincer_1_joint" type="fixed">
+            <parent link="${prefix}schunk_egp50_body_link" />
+            <child link="${prefix}schunk_egp50_pincer_1_link" />
             <origin xyz="0.0 0.0 ${body_height/2+pincer_height/2}" rpy="0.0 0.0 0.0" />
             <!-- the motion of the pincer is along the X axis -->
@@ -114,7 +119,7 @@
             <limit lower="${-body_length/16}" upper="${body_length/16}" velocity="100" effort="100" />
         </joint>
-        <joint name="shunk_egp50_pincer_2_joint" type="fixed">
-            <parent link="shunk_egp50_body_link" />
-            <child link="shunk_egp50_pincer_2_link" />
+        <joint name="schunk_egp50_pincer_2_joint" type="fixed">
+            <parent link="${prefix}schunk_egp50_body_link" />
+            <child link="${prefix}schunk_egp50_pincer_2_link" />
             <origin xyz="0.0 0.002 ${body_height/2+pincer_height/2}" rpy="0.0 0.0 0.0" />
             <!-- the motion of the pincer is along the X axis -->
@@ -123,9 +128,17 @@
             <limit lower="${body_length/16}" upper="${-body_length/16}" velocity="100" effort="100" />
         </joint>
-        <joint name="shunk_egp50_tip_joint" type="fixed">
-            <parent link="shunk_egp50_base_link" />
+        <joint name="${prefix}schunk_egp50_tip_joint" type="fixed">
+            <parent link="${prefix}schunk_egp50_base_link" />
             <child link="tool_tip" />
             <origin xyz="0 0 ${body_height_max}" rpy="0.0 0.0 0.0" />
         </joint>
+        <joint
+            name="schunk_egp50_base_joint"
+            type="fixed"
+        >
+            <parent link="${parent}" />
+            <child link="${prefix}schunk_egp50_base_link" />
+            <xacro:insert_block name="origin" />
+        </joint>
     </xacro:macro>
 </robot>

File: ur5e_cell_description/urdf/workcell.urdf.xacro (robot description, xacro)
@@ -4,5 +4,5 @@
     <xacro:include filename="$(find ur5e_cell_description)/urdf/robot_cell.xacro" />
     <!-- inlcuding components for loading xacros -->
-    <xacro:include filename="$(find ur5e_cell_description)/urdf/shunk_egp50.xacro" />
+    <xacro:include filename="$(find ur5e_cell_description)/urdf/schunk_egp50.xacro" />
     <xacro:include filename="$(find ur_description)/urdf/ur_macro.xacro" />
     <xacro:include filename="$(find realsense2_description)/urdf/_d435.urdf.xacro" />
@@ -41,8 +41,16 @@
     <!-- Set arg initial_positions_file as property -->
     <xacro:property name="initial_positions_file" default="$(arg initial_positions_file)" />
-    <!-- Args related to realsense
+    <!-- Args related to realsense -->
     <xacro:arg name="use_nominal_extrinsics" default="false"/>
     <xacro:arg name="add_plug" default="false" />
-    <xacro:arg name="use_mesh" default="true" /> -->
+    <xacro:arg name="use_mesh" default="true" />
+    <!-- Add world link -->
+    <link name="world" />
+    <xacro:robot_cell
+      name="robot_cell"
+      prefix=""
+      parent="world">
+    <origin xyz="0 0 0" rpy="0 0 0" />
+    </xacro:robot_cell>
     <!-- Robot cell is directly included from its xacro as it is no macro. -->
     <!-- Instantiate UR robot. -->
@@ -50,5 +58,5 @@
         name="$(arg name)"
         prefix="$(arg prefix)"
-        parent="robotcell_base_link"
+        parent="robot_link"
         joint_limits_parameters_file="$(arg joint_limit_params)"
         kinematics_parameters_file="$(arg kinematics_params)"
@@ -79,10 +87,15 @@
         input_recipe_filename="$(arg input_recipe_filename)"
     >
-        <origin xyz="${robot_center_offset_length} ${robot_center_offset_width} ${robot_base_height}" rpy="0 0 ${pi/2}" /> <!-- position robot in the world -->
+        <origin xyz="0 0 0" rpy="0 0 ${pi/2}" />
     </xacro:ur_robot>
     <!-- Instantiate gripper. -->
-    <xacro:schunk_egp50 />
+    <xacro:schunk_egp50
+      parent="tool0"
+      name="schunk_egp50"
+      prefix="">
+      <origin xyz="0 0 0" rpy="0 0 0" />
+    </xacro:schunk_egp50>
     <!-- Instantiate camera. -->
-    <!-- <xacro:sensor_d435
+    <xacro:sensor_d435
         parent="tool0"
         use_nominal_extrinsics="$(arg use_nominal_extrinsics)"
@@ -90,25 +103,26 @@
         use_mesh="$(arg use_mesh)"
     >
-        <origin xyz="0 -0.05 0" rpy="${pi/2} ${pi/2} 0"/>
-    </xacro:sensor_d435> -->
-    <!-- Add world link -->
-    <link name="world" />
-    <!-- Add joint between robotcell and world -->
-    <joint
-        name="world_to_robot_cell_joint"
-        type="fixed"
-    >
-        <parent link="world" />
-        <child link="robotcell_base_link" />
-        <origin xyz="0 0 0" rpy="0 0 0" />
-    </joint>
-    <!-- Add joint between gripper and robot -->
-    <joint
-        name="robot_to_gripper_joint"
-        type="fixed"
-    >
-        <parent link="tool0" />
-        <child link="shunk_egp50_base_link" />
-        <origin xyz="0 0 0" rpy="0 0 0" />
-    </joint>
+        <origin xyz="0 -0.05 0" rpy="${pi/2} -${pi/2} 0"/>
+    </xacro:sensor_d435>
+   <xacro:if value="$(arg sim_gazebo)">
+    <!-- Gazebo plugins -->
+    <gazebo reference="world">
+    </gazebo>
+    <gazebo>
+      <plugin filename="libgazebo_ros2_control.so" name="gazebo_ros2_control">
+        <parameters>$(arg simulation_controllers)</parameters>
+      </plugin>
+    </gazebo>
+  </xacro:if>
+  <xacro:if value="$(arg sim_ignition)">
+    <!-- Gazebo plugins -->
+    <gazebo reference="world">
+    </gazebo>
+    <gazebo>
+      <plugin filename="libign_ros2_control-system.so" name="ign_ros2_control::IgnitionROS2ControlPlugin">
+        <parameters>$(arg simulation_controllers)</parameters>
+        <controller_manager_node_name>$(arg prefix)controller_manager</controller_manager_node_name>
+      </plugin>
+    </gazebo>
+  </xacro:if>
 </robot>
