Commit message: change "prefix" to "tf_prefix"

File: ur5e_cell_description/urdf/robot_cell.xacro (robot description, xacro)
@@ -4,5 +4,5 @@
     <xacro:macro name="robot_cell" params="
         name
-        prefix
+        tf_prefix
         parent
         *origin">
@@ -17,5 +17,5 @@
             <color rgba="0.6 0.8 0.8 1" />
         </material>
-        <link name="${prefix}visuals_link">
+        <link name="${tf_prefix}visuals_link">
             <visual>
                 <geometry>
@@ -25,5 +25,5 @@
             </visual>
         </link>
-        <link name="${prefix}shield_front_link">
+        <link name="${tf_prefix}shield_front_link">
             <collision>
                 <origin rpy="0 0 0" xyz="0 0 0" />
@@ -37,5 +37,5 @@
             </xacro:inertial_box>
         </link>
-        <link name="${prefix}shield_rear_link">
+        <link name="${tf_prefix}shield_rear_link">
             <collision>
                 <origin rpy="0 0 0 " xyz="0 0 0" />
@@ -49,5 +49,5 @@
             </xacro:inertial_box>
         </link>
-        <link name="${prefix}shield_right_link">
+        <link name="${tf_prefix}shield_right_link">
             <collision>
                 <origin rpy="0 0 0" xyz="0 0 0" />
@@ -61,5 +61,5 @@
             </xacro:inertial_box>
         </link>
-        <link name="${prefix}shield_left_link">
+        <link name="${tf_prefix}shield_left_link">
             <collision>
                 <origin rpy="0 0 0" xyz="0 0 0" />
@@ -73,5 +73,5 @@
             </xacro:inertial_box>
         </link>
-        <link name="${prefix}robotcell_base_link">
+        <link name="${tf_prefix}robotcell_base_link">
             <collision>
                 <origin rpy="0 0 0" xyz="0 0 ${robot_base_height/2}" />
@@ -85,38 +85,38 @@
             </xacro:inertial_box>
         </link>
-        <link name="${prefix}robot_link" />
-        <joint name="${prefix}robotcell_base_to_visual" type="fixed">
-            <parent link="${prefix}robotcell_base_link" />
-            <child link="${prefix}visuals_link" />
+        <link name="${tf_prefix}robot_link" />
+        <joint name="${tf_prefix}robotcell_base_to_visual" type="fixed">
+            <parent link="${tf_prefix}robotcell_base_link" />
+            <child link="${tf_prefix}visuals_link" />
             <origin xyz="${robotcell_length/2+shield_thickness} -${robotcell_width/2+shield_thickness} 0" rpy="0 0 ${pi/2}" />
         </joint>
-        <joint name="${prefix}robotcell_base_to_front_joint" type="fixed">
-            <parent link="${prefix}robotcell_base_link" />
-            <child link="${prefix}shield_front_link" />
+        <joint name="${tf_prefix}robotcell_base_to_front_joint" type="fixed">
+            <parent link="${tf_prefix}robotcell_base_link" />
+            <child link="${tf_prefix}shield_front_link" />
             <origin xyz="0 ${robotcell_width/2-shield_thickness/2} ${robot_base_height+robotcell_height/2}" rpy="0 0 0" />
         </joint>
-        <joint name="${prefix}robotcell_base_to_rear" type="fixed">
-            <parent link="${prefix}robotcell_base_link" />
-            <child link="${prefix}shield_rear_link" />
+        <joint name="${tf_prefix}robotcell_base_to_rear" type="fixed">
+            <parent link="${tf_prefix}robotcell_base_link" />
+            <child link="${tf_prefix}shield_rear_link" />
             <origin xyz="0 ${-robotcell_width/2+shield_thickness/2} ${robot_base_height+robotcell_height/2}" rpy="0 0 0" />
         </joint>
-        <joint name="${prefix}robotcell_base_to_left" type="fixed">
-            <parent link="${prefix}robotcell_base_link" />
-            <child link="${prefix}shield_left_link" />
+        <joint name="${tf_prefix}robotcell_base_to_left" type="fixed">
+            <parent link="${tf_prefix}robotcell_base_link" />
+            <child link="${tf_prefix}shield_left_link" />
             <origin xyz="${-robotcell_length/2+shield_thickness/2} 0 ${robot_base_height+robotcell_height/2}" rpy="0 0 0" />
         </joint>
-        <joint name="${prefix}robotcell_base_to_right" type="fixed">
-            <parent link="${prefix}robotcell_base_link" />
-            <child link="${prefix}shield_right_link" />
+        <joint name="${tf_prefix}robotcell_base_to_right" type="fixed">
+            <parent link="${tf_prefix}robotcell_base_link" />
+            <child link="${tf_prefix}shield_right_link" />
             <origin xyz="${robotcell_length/2-shield_thickness/2} 0 ${robot_base_height+robotcell_height/2}" rpy="0 0 0" />
         </joint>
-        <joint name="${prefix}robot_cell_base_joint" type="fixed">
+        <joint name="${tf_prefix}robot_cell_base_joint" type="fixed">
             <parent link="${parent}" />
-            <child link="${prefix}robotcell_base_link" />
+            <child link="${tf_prefix}robotcell_base_link" />
             <xacro:insert_block name="origin" />
         </joint>
-        <joint name="${prefix}robot_cell_base_to_robot_link" type="fixed">
-            <parent link="${prefix}robotcell_base_link" />
-            <child link="${prefix}robot_link" />
+        <joint name="${tf_prefix}robot_cell_base_to_robot_link" type="fixed">
+            <parent link="${tf_prefix}robotcell_base_link" />
+            <child link="${tf_prefix}robot_link" />
             <origin xyz="${robot_center_offset_length} ${robot_center_offset_width} ${robot_base_height}" rpy="0 0 0" />
         </joint>

File: ur5e_cell_description/urdf/workcell.urdf.xacro (robot description, xacro)
@@ -10,5 +10,5 @@
     <xacro:arg name="name" default="ur5e" />
     <xacro:arg name="ur_type" default="ur5e" />
-    <xacro:arg name="prefix" default="" />
+    <xacro:arg name="tf_prefix" default="" />
     <xacro:arg name="joint_limit_params" default="$(find ur5e_cell_description)/config/$(arg ur_type)/joint_limits.yaml" />
     <xacro:arg name="kinematics_params" default="$(find ur5e_cell_description)/config/$(arg ur_type)/default_kinematics.yaml" />
@@ -49,5 +49,5 @@
     <xacro:robot_cell
       name="robot_cell"
-      prefix=""
+      tf_prefix=""
       parent="world">
     <origin xyz="0 0 0" rpy="0 0 0" />
@@ -57,5 +57,5 @@
     <xacro:ur_robot
         name="$(arg name)"
-        prefix="$(arg prefix)"
+        tf_prefix="$(arg tf_prefix)"
         parent="robot_link"
         joint_limits_parameters_file="$(arg joint_limit_params)"

File: ur5e_cell_moveit_config/config/ur5e_workcell.urdf.xacro (robot description, xacro)
@@ -4,5 +4,5 @@
     <xacro:arg name="name" default="ur5e_workcell" />
     <xacro:arg name="ur_type" default="ur5e" />
-    <xacro:arg name="prefix" default="" />
+    <xacro:arg name="tf_prefix" default="" />
     <xacro:arg name="script_filename" default="$(find ur_robot_driver)/resources/ros_control.urscript" />
     <xacro:arg name="output_recipe_filename" default="$(find ur_robot_driver)/resources/rtde_output_recipe.txt" />
@@ -11,5 +11,5 @@
     <xacro:arg name="fake_sensor_commands" default="true" />
     <xacro:arg name="robot_ip" default="192.168.56.2" />
-    <xacro:arg name="prefix" default="" />
+    <xacro:arg name="tf_prefix" default="" />
     <!-- Import ur5e_workcell urdf file -->
     <xacro:include filename="$(find ur5e_cell_description)/urdf/workcell.urdf.xacro" />
